File: outputs/pcbs/main_pcb.kicad_pcb (KiCad board)
At the start: 2 copper layers, 161.7 x 111.9 mm, 85 parts

Commit message: 22d
Connections:
- net k_0_r_0_DIN renamed D0
- net k_0_r_3_DOUT renamed D28
- LED1 pad 4: k_0_r_3_DIN -> D27
- LED10 pad 2: k_2_r_2_DOUT -> D14
- LED10 pad 4: k_2_r_2_DIN -> D13
- LED11 pad 2: k_2_r_1_DOUT -> D9
- LED11 pad 4: k_2_r_1_DIN -> D8
- LED12 pad 2: k_2_r_0_DOUT -> D3
- LED12 pad 4: k_2_r_0_DIN -> D2
- LED13 pad 2: k_3_r_3_DOUT -> D25
- LED13 pad 4: k_3_r_3_DIN -> D24
- LED14 pad 2: k_3_r_2_DOUT -> D15
- LED14 pad 4: k_3_r_2_DIN -> D14
- LED15 pad 2: k_3_r_1_DOUT -> D8
- LED15 pad 4: k_3_r_1_DIN -> D7
- LED16 pad 2: k_3_r_0_DOUT -> D4
- LED16 pad 4: k_3_r_0_DIN -> D3
- LED17 pad 2: k_4_r_3_DOUT -> D24
- LED17 pad 4: k_4_r_3_DIN -> D23
- LED18 pad 2: k_4_r_2_DOUT -> D16
- LED18 pad 4: k_4_r_2_DIN -> D15
- LED19 pad 2: k_4_r_1_DOUT -> D7
- LED19 pad 4: k_4_r_1_DIN -> D6
- LED2 pad 2: k_0_r_2_DOUT -> D12
- LED2 pad 4: k_0_r_2_DIN -> D11
- LED20 pad 2: k_4_r_0_DOUT -> D5
- LED20 pad 4: k_4_r_0_DIN -> D4
- LED21 pad 2: k_5_r_2_DOUT -> D17
- LED21 pad 4: k_5_r_2_DIN -> D16
- LED22 pad 2: k_5_r_1_DOUT -> D6
- LED22 pad 4: k_5_r_1_DIN -> D5
- LED23 pad 2: t1_td_DOUT -> D18
- LED23 pad 4: t1_td_DIN -> D17
- LED24 pad 2: t1_tu_DOUT -> D23
- LED24 pad 4: t1_tu_DIN -> D22
- LED25 pad 2: t2_td_DOUT -> D19
- LED25 pad 4: t2_td_DIN -> D18
- LED26 pad 2: t2_tu_DOUT -> D22
- LED26 pad 4: t2_tu_DIN -> D21
- LED27 pad 2: t3_td_DOUT -> D20
- LED27 pad 4: t3_td_DIN -> D19
- LED28 pad 2: t3_tu_DOUT -> D21
- LED28 pad 4: t3_tu_DIN -> D20
- LED3 pad 2: k_0_r_1_DOUT -> D11
- LED3 pad 4: k_0_r_1_DIN -> D10
- LED4 pad 2: k_0_r_0_DOUT -> D1
- LED5 pad 2: k_1_r_3_DOUT -> D27
- LED5 pad 4: k_1_r_3_DIN -> D26
- LED6 pad 2: k_1_r_2_DOUT -> D13
- LED6 pad 4: k_1_r_2_DIN -> D12
- LED7 pad 2: k_1_r_1_DOUT -> D10
- LED7 pad 4: k_1_r_1_DIN -> D9
- LED8 pad 2: k_1_r_0_DOUT -> D2
- LED8 pad 4: k_1_r_0_DIN -> D1
- LED9 pad 2: k_2_r_3_DOUT -> D26
- LED9 pad 4: k_2_r_3_DIN -> D25
Routing:
- net D24: track 0.00 -> 13.5 mm, vias 0 -> 2
- net D9: track 0.00 -> 13.5 mm, vias 0 -> 2
- net D23: track 0.00 -> 13.5 mm, vias 0 -> 2
- net D5: track 0.00 -> 13.5 mm, vias 0 -> 2
- net D14: track 0.00 -> 13.5 mm, vias 0 -> 2
- net D8: track 0.00 -> 13.5 mm, vias 0 -> 2
- net D13: track 0.00 -> 13.5 mm, vias 0 -> 2
- net D1: track 0.00 -> 13.5 mm, vias 0 -> 2
- net D2: track 0.00 -> 13.5 mm, vias 0 -> 2
- net D17: track 0.00 -> 13.5 mm, vias 0 -> 2
- net D16: track 0.00 -> 13.5 mm, vias 0 -> 2
- net D21: track 0.00 -> 13.5 mm, vias 0 -> 2
- net D15: track 0.00 -> 13.5 mm, vias 0 -> 2
- net D3: track 0.00 -> 13.5 mm, vias 0 -> 2
- net D6: track 0.00 -> 13.5 mm, vias 0 -> 2
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
Commit message: cpu added
Parts:
- moved REF** 97.0 mm to (85.0, 41.2), turned to 1 degrees
Connections:
- REF** pad 1: (no net) -> VCC
- REF** pad 10: (no net) -> t_2
- REF** pad 11: (no net) -> K_5
- REF** pad 12: (no net) -> K_4
- REF** pad 13: (no net) -> K_3
- REF** pad 14: (no net) -> K_2
- REF** pad 15: (no net) -> K_1
- REF** pad 16: (no net) -> K_0
- REF** pad 17: (no net) -> R_0
- REF** pad 18: (no net) -> R_1
- REF** pad 2: (no net) -> GND
- REF** pad 22: (no net) -> R_3
- REF** pad 23: (no net) -> R_2
Other:
- board size 161.7 x 111.9 mm -> 163.7 x 126 mm

Commit message: 1
Parts:
- moved REF** 14.9 mm to (99.6, 38.6), turned to 5 degrees
Other:
- board size 163.7 x 126 mm -> 163.7 x 129 mm

Commit message: parts
Parts:
- added REF**: Jack_3.5mm_PJ320E_Horizontal, Connector_Audio:Jack_3.5mm_PJ320E_Horizontal, F.Cu at (158.8, 40.7)
- moved REF** 0.28 mm to (99.8, 38.8)
Other:
- board size 163.7 x 129 mm -> 162.5 x 128.8 mm

Commit message: all good1
Parts:
- added REF**: PinHeader_1x05_P2.54mm_Vertical, Connector_PinHeader_2.54mm:PinHeader_1x05_P2.54mm_Vertical, F.Cu at (76.5, 54.8)
- added REF**: R_0805_2012Metric_Pad1.20x1.40mm_HandSolder, Resistor_SMD:R_0805_2012Metric_Pad1.20x1.40mm_HandSolder, F.Cu at (88.1, 53.0)
- added REF**: R_0805_2012Metric_Pad1.20x1.40mm_HandSolder, Resistor_SMD:R_0805_2012Metric_Pad1.20x1.40mm_HandSolder, F.Cu at (84.4, 51.4)
Connections:
- REF** pad 10: t_2 -> cross_board
- REF** pad 20: (no net) -> D0
- REF** pad 21: (no net) -> t_2
- REF** pad 3: (no net) -> 3v3
- REF** pad 8: (no net) -> gp15
- REF** pad 9: (no net) -> gp14
- REF** pad R1: (no net) -> cross_board
- REF** pad R2: (no net) -> GND
- REF** pad S: (no net) -> GND
- REF** pad T: (no net) -> VCC
Other:
- board size 162.5 x 128.8 mm -> 162 x 128.8 mm
- board text added: "5 GND 3v3 14 15"

Commit message: different nets
Parts:
- moved REF** 5.12 mm to (88.5, 47.9)
- moved REF** 4.18 mm to (77.8, 50.8)
- moved REF** 1.68 mm to (86.0, 51.9)
Connections:
- REF** pad 11: K_5 -> K_2
- REF** pad 12: K_4 -> K_1
- REF** pad 13: K_3 -> K_0
- REF** pad 15: K_1 -> R_3
- REF** pad 16: K_0 -> R_2
- REF** pad 17: R_0 -> R_1
- REF** pad 18: R_1 -> R_0
- REF** pad 19: (no net) -> t_2
- REF** pad 20: D0 -> K_5
- REF** pad 21: t_2 -> K_4
- REF** pad 22: R_3 -> K_3
- REF** pad 23: R_2 -> D0
Other:
- board size 162 x 128.8 mm -> 166.5 x 128.8 mm

Commit message: routing1
Connections:
- REF** pad 15: R_3 -> R_0
- REF** pad 16: R_2 -> R_1
- REF** pad 17: R_1 -> R_2
- REF** pad 18: R_0 -> R_3
Routing:
- net R_0: track 0.00 -> 251.5 mm, vias 0 -> 7
- net R_1: track 0.00 -> 246.1 mm, vias 0 -> 9
- net R_3: track 0.00 -> 205.4 mm, vias 0 -> 7
- net t_2: track 33.1 -> 215.8 mm, vias 4 -> 5
- net K_5: track 33.1 -> 214.3 mm, vias 4 -> 6
- net R_2: track 0.00 -> 180.2 mm, vias 0 -> 7
- net K_4: track 33.1 -> 161.4 mm, vias 4 -> 7
- net GND: track 105.1 -> 17.5 mm, vias 28 -> 3
- net VCC: track 105.1 -> 26.6 mm, vias 28 -> 2
- net cross_board: track 0.00 -> 64.4 mm
- net K_1: track 33.1 -> 94.5 mm
- net K_3: track 33.1 -> 91.5 mm
- net K_2: track 33.1 -> 89.4 mm
- net K_0: track 33.1 -> 81.4 mm
- net D17: track 13.5 -> 58.1 mm
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- added copper zone on B.Cu, net GND
- added copper zone on F.Cu, net VCC

Commit message: routing2
Connections:
- REF** pad 11: K_2 -> (no net)
Routing:
- net K_3: track 91.5 -> 262.8 mm, vias 4 -> 7
- net K_0: track 81.4 -> 171.0 mm, vias 4 -> 7
- net VCC: track 26.6 -> 104.9 mm, vias 2 -> 30
- net K_1: track 94.5 -> 144.9 mm, vias 4 -> 7
- net D22: track 8.17 -> 53.8 mm, vias 1 -> 2
- net R_2: track 180.2 -> 218.7 mm
- net GND: track 17.5 -> 53.8 mm, vias 3 -> 29
- net D0: track 3.92 -> 38.7 mm, vias 1 -> 2
- net K_2: track 89.4 -> 117.6 mm, vias 4 -> 5
- net gp15: track 0.00 -> 11.1 mm
- net 3v3: track 24.0 -> 31.9 mm
- net D21: track 50.4 -> 57.7 mm, vias 2 -> 3
- net t2_tu: track 36.1 -> 41.4 mm
- net K_4: track 161.4 -> 166.2 mm
- net D24: track 39.1 -> 37.8 mm
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