File: outputs/pcbs/main_pcb.kicad_pcb (KiCad board)
At the start: 2 copper layers, 166.5 x 128.8 mm, 89 parts

Commit message: routing3
Routing:
- net VCC: track 104.9 -> 168.9 mm, vias 30 -> 38
- net t_2: track 215.8 -> 239.2 mm, vias 5 -> 8
- net GND: track 53.8 -> 70.3 mm, vias 29 -> 33
- net t2_td: track 29.0 -> 37.0 mm
- net R_1: track 246.1 -> 249.4 mm, vias 9 -> 10
- net D11: track 36.1 -> 32.9 mm
- net D6: track 40.7 -> 38.0 mm, vias 2 -> 3
- net D24: track 37.8 -> 39.9 mm, vias 3 -> 5
- net D10: track 39.1 -> 38.2 mm
- net K_0: track 171.0 -> 171.7 mm, vias 7 -> 6
Other:
- board size 166.5 x 128.8 mm -> 163.5 x 128.8 mm

Commit message: all connected all good
Routing:
- net VCC: track 168.9 -> 304.5 mm, vias 38 -> 60
- net GND: track 70.3 -> 201.2 mm, vias 33 -> 53
- net gp14: track 7.16 -> 15.4 mm
- net t3_td: track 27.3 -> 34.9 mm, vias 0 -> 1
- net D8: track 40.6 -> 44.0 mm, vias 3 -> 4
- net D25: track 36.8 -> 39.6 mm
- net D15: track 22.1 -> 24.4 mm
- net D10: track 38.2 -> 40.4 mm
- net K_3: track 262.5 -> 264.4 mm
- net D3: track 24.4 -> 25.9 mm
- net D9: track 37.4 -> 38.8 mm
- net D26: track 40.5 -> 41.7 mm
- net D7: track 37.5 -> 38.6 mm
- net D2: track 23.4 -> 24.4 mm
- net 3v3: track 31.9 -> 32.8 mm, vias 1 -> 2
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